Commit message: added option for minimal collisions

File: talos_description/urdf/arm/arm.urdf.xacro (robot description, xacro)
@@ -24,5 +24,5 @@
   <xacro:property name="arm_4_max_effort"   value="70.0" />
   <xacro:property name="arm_eps"            value="0.02" />
-  <xacro:macro name="talos_arm" params="name parent side reflect">
+  <xacro:macro name="talos_arm" params="name parent side reflect minimal_coll:=false">
     <xacro:unless value="$(arg test)">
       <xacro:include filename="${TALOS_DESCRIPTION_CALIBRATION_ROOT}/urdf/calibration/arm_${side}.xacro" />
@@ -43,14 +43,16 @@
         <material name="DarkGrey" />
       </visual>
-      <xacro:if value="$(arg use_capsule_collision)">
-        <xacro:capsule-collision e1="-0.030119 0.141768 0.0465263" e2="-0.00429634 0.0157203 0.0513477" rad="0.076661652397679497" clen="0.12875612953621868" rpy="1.53256 0.201924 0.194397" mid="-0.0172077 0.0787443 0.048937" reflect="${reflect}" />
-      </xacro:if>
-      <xacro:unless value="$(arg use_capsule_collision)">
-        <collision>
-          <origin xyz="0 0 0" rpy="0 0 0" />
-          <geometry>
-            <mesh filename="${MESH_PATH}/arm/arm_1_collision.STL" scale="1 ${reflect} 1"/>
-          </geometry>
-        </collision>
+      <xacro:unless value="${minimal_coll}">
+        <xacro:if value="$(arg use_capsule_collision)">
+          <xacro:capsule-collision e1="-0.030119 0.141768 0.0465263" e2="-0.00429634 0.0157203 0.0513477" rad="0.076661652397679497" clen="0.12875612953621868" rpy="1.53256 0.201924 0.194397" mid="-0.0172077 0.0787443 0.048937" reflect="${reflect}" />
+        </xacro:if>
+        <xacro:unless value="$(arg use_capsule_collision)">
+          <collision>
+            <origin xyz="0 0 0" rpy="0 0 0" />
+            <geometry>
+              <mesh filename="${MESH_PATH}/arm/arm_1_collision.STL" scale="1 ${reflect} 1"/>
+            </geometry>
+          </collision>
+        </xacro:unless>
       </xacro:unless>
     </link>
@@ -111,14 +113,16 @@
         <material name="DarkGrey" />
       </visual>
-      <xacro:if value="$(arg use_capsule_collision)">
-        <xacro:capsule-collision e1="0.0012938 0.00577828 -0.203827" e2="0.0206547 0.0332832 -0.277413" rad="0.077010074599207598" clen="0.080908820017687497" rpy="-2.78389 0.241638 -1.1828" mid="0.0109743 0.0195307 -0.24062" reflect="${reflect}" />
-      </xacro:if>
-      <xacro:unless value="$(arg use_capsule_collision)">
-        <collision>
-          <origin xyz="0 0 0" rpy="0 0 0" />
-          <geometry>
-            <mesh filename="${MESH_PATH}/arm/arm_3_collision.STL" scale="1 ${reflect} 1"/>
-          </geometry>
-        </collision>
+      <xacro:unless value="${minimal_coll}">
+        <xacro:if value="$(arg use_capsule_collision)">
+          <xacro:capsule-collision e1="0.0012938 0.00577828 -0.203827" e2="0.0206547 0.0332832 -0.277413" rad="0.077010074599207598" clen="0.080908820017687497" rpy="-2.78389 0.241638 -1.1828" mid="0.0109743 0.0195307 -0.24062" reflect="${reflect}" />
+        </xacro:if>
+        <xacro:unless value="$(arg use_capsule_collision)">
+          <collision>
+            <origin xyz="0 0 0" rpy="0 0 0" />
+            <geometry>
+              <mesh filename="${MESH_PATH}/arm/arm_3_collision.STL" scale="1 ${reflect} 1"/>
+            </geometry>
+          </collision>
+        </xacro:unless>
       </xacro:unless>
     </link>
@@ -208,5 +212,5 @@
     <!--        WRIST           -->
     <!--************************-->
-    <xacro:talos_wrist name="arm" parent="${name}_${side}_4_link" side="${side}" reflect="${reflect}" />
+    <xacro:talos_wrist name="arm" parent="${name}_${side}_4_link" side="${side}" reflect="${reflect}" minimal_coll="${minimal_coll}" />
   </xacro:macro>
 </robot>

File: talos_description/urdf/arm/wrist.urdf.xacro (robot description, xacro)
@@ -21,5 +21,5 @@
   <xacro:property name="wrist_3_max_effort"   value="8.0" />
   <xacro:property name="wrist_eps"          value="0.02" />
-  <xacro:macro name="talos_wrist" params="name parent side reflect">
+  <xacro:macro name="talos_wrist" params="name parent side reflect minimal_coll:=false">
     <xacro:unless value="$(arg test)">
       <xacro:include filename="${TALOS_DESCRIPTION_CALIBRATION_ROOT}/urdf/calibration/arm_${side}.xacro" />
@@ -40,14 +40,16 @@
         <material name="LightGrey" />
       </visual>
-      <xacro:if value="$(arg use_capsule_collision)">
-        <xacro:capsule-collision e1="-2.13964e-05 0.000999035 0.0358616" e2="0.000145615 0.0012191 0.121451" rad="0.077412213480368891" clen="0.085589949413547098" rpy="-0.00257122 0.0019513 -2.50861e-06" mid="6.21094e-05 0.00110907 0.0786563" reflect="${reflect}" />
-      </xacro:if>
-      <xacro:unless value="$(arg use_capsule_collision)">
-        <collision>
-          <origin xyz="0 0 0" rpy="0 0 0" />
-          <geometry>
-            <mesh filename="${MESH_PATH}/arm/arm_5_collision.STL" scale="1 ${reflect} 1"/>
-          </geometry>
-        </collision>
+      <xacro:unless value="${minimal_coll}">
+        <xacro:if value="$(arg use_capsule_collision)">
+          <xacro:capsule-collision e1="-2.13964e-05 0.000999035 0.0358616" e2="0.000145615 0.0012191 0.121451" rad="0.077412213480368891" clen="0.085589949413547098" rpy="-0.00257122 0.0019513 -2.50861e-06" mid="6.21094e-05 0.00110907 0.0786563" reflect="${reflect}" />
+        </xacro:if>
+        <xacro:unless value="$(arg use_capsule_collision)">
+          <collision>
+            <origin xyz="0 0 0" rpy="0 0 0" />
+            <geometry>
+              <mesh filename="${MESH_PATH}/arm/arm_5_collision.STL" scale="1 ${reflect} 1"/>
+            </geometry>
+          </collision>
+        </xacro:unless>
       </xacro:unless>
     </link>
@@ -74,14 +76,16 @@
         <material name="LightGrey" />
       </visual>
-      <xacro:if value="$(arg use_capsule_collision)">
-        <xacro:capsule-collision e1="3.71733e-07 -0.000248227 -0.00766634" e2="5.46154e-05 -8.61821e-05 0.00107298" rad="0.044402592090813625" clen="0.0087409825962203314" rpy="-0.0185399 0.00620572 -5.75286e-05" mid="2.74936e-05 -0.000167204 -0.00329668" reflect="${reflect}" />
-      </xacro:if>
-      <xacro:unless value="$(arg use_capsule_collision)">
-        <collision>
-          <origin xyz="0 0 0" rpy="0 0 0" />
-          <geometry>
-            <mesh filename="${MESH_PATH}/arm/arm_6_collision.STL" scale="1 ${reflect} 1"/>
-          </geometry>
-        </collision>
+      <xacro:unless value="${minimal_coll}">
+        <xacro:if value="$(arg use_capsule_collision)">
+          <xacro:capsule-collision e1="3.71733e-07 -0.000248227 -0.00766634" e2="5.46154e-05 -8.61821e-05 0.00107298" rad="0.044402592090813625" clen="0.0087409825962203314" rpy="-0.0185399 0.00620572 -5.75286e-05" mid="2.74936e-05 -0.000167204 -0.00329668" reflect="${reflect}" />
+        </xacro:if>
+        <xacro:unless value="$(arg use_capsule_collision)">
+          <collision>
+            <origin xyz="0 0 0" rpy="0 0 0" />
+            <geometry>
+              <mesh filename="${MESH_PATH}/arm/arm_6_collision.STL" scale="1 ${reflect} 1"/>
+            </geometry>
+          </collision>
+        </xacro:unless>
       </xacro:unless>
     </link>

File: talos_description/urdf/head/head.urdf.xacro (robot description, xacro)
@@ -32,14 +32,16 @@
         <material name="DarkGrey" />
       </visual>
-      <xacro:if value="$(arg use_capsule_collision)">
-        <xacro:capsule-collision e1="9.25184e-05 -2.39435e-05 -0.000765958" e2="-0.0116532 0.000267479 0.0600432" rad="0.082632032931063207" clen="0.061933815385056032" rpy="-0.00479238 -0.190806 0.000458601" mid="-0.00578036 0.000121768 0.0296386" />
-      </xacro:if>
-      <xacro:unless value="$(arg use_capsule_collision)">
-        <collision>
-          <origin xyz="0 0 0" rpy="0 0 0" />
-          <geometry>
-            <mesh filename="${MESH_PATH}/head/head_1_collision.stl" scale="1 1 1"/>
-          </geometry>
-        </collision>
+      <xacro:unless value="$(arg minimal_coll)">
+        <xacro:if value="$(arg use_capsule_collision)">
+          <xacro:capsule-collision e1="9.25184e-05 -2.39435e-05 -0.000765958" e2="-0.0116532 0.000267479 0.0600432" rad="0.082632032931063207" clen="0.061933815385056032" rpy="-0.00479238 -0.190806 0.000458601" mid="-0.00578036 0.000121768 0.0296386" />
+        </xacro:if>
+        <xacro:unless value="$(arg use_capsule_collision)">
+          <collision>
+            <origin xyz="0 0 0" rpy="0 0 0" />
+            <geometry>
+              <mesh filename="${MESH_PATH}/head/head_1_collision.stl" scale="1 1 1"/>
+            </geometry>
+          </collision>
+        </xacro:unless>
       </xacro:unless>
     </link>
@@ -81,14 +83,16 @@
         <material name="LightGrey" />
       </visual>
-      <xacro:if value="$(arg use_capsule_collision)">
-        <xacro:capsule-collision e1="-0.0136558 6.17209e-05 0.196249" e2="0.0257541 0.000121936 0.169493" rad="0.10582827877003444" clen="0.047634451110799531" rpy="-3.13934 0.974356 -3.13734" mid="0.00604916 9.18284e-05 0.182871" />
-      </xacro:if>
-      <xacro:unless value="$(arg use_capsule_collision)">
-        <collision>
-          <origin xyz="0 0 0" rpy="0 0 0" />
-          <geometry>
-            <mesh filename="${MESH_PATH}/head/head_2_${type}_collision.stl" scale="1 1 1"/>
-          </geometry>
-        </collision>
+      <xacro:unless value="$(arg minimal_coll)">
+        <xacro:if value="$(arg use_capsule_collision)">
+          <xacro:capsule-collision e1="-0.0136558 6.17209e-05 0.196249" e2="0.0257541 0.000121936 0.169493" rad="0.10582827877003444" clen="0.047634451110799531" rpy="-3.13934 0.974356 -3.13734" mid="0.00604916 9.18284e-05 0.182871" />
+        </xacro:if>
+        <xacro:unless value="$(arg use_capsule_collision)">
+          <collision>
+            <origin xyz="0 0 0" rpy="0 0 0" />
+            <geometry>
+              <mesh filename="${MESH_PATH}/head/head_2_${type}_collision.stl" scale="1 1 1"/>
+            </geometry>
+          </collision>
+        </xacro:unless>
       </xacro:unless>
     </link>

File: talos_description/urdf/leg/leg.urdf.xacro (robot description, xacro)
@@ -7,5 +7,5 @@
   <xacro:property name="leg_friction"     value="0.0" />
   <xacro:property name="leg_damping"      value="0.0" />
-  <xacro:macro name="talos_leg" params="prefix reflect flexibility:=false">
+  <xacro:macro name="talos_leg" params="prefix reflect flexibility:=false minimal_coll:=false">
     <xacro:unless value="$(arg test)">
       <xacro:include filename="${TALOS_DESCRIPTION_CALIBRATION_ROOT}/urdf/calibration/leg_${prefix}.xacro" />
@@ -71,14 +71,16 @@
         <material name="DarkGrey" />
       </visual>
-      <xacro:if value="$(arg use_capsule_collision)">
-        <xacro:capsule-collision e1="0.00653137 -0.00107636 0.0620231" e2="0.0148595 0.000151801 0.00431736" rad="0.10038884516307987" clen="0.058316498699378369" rpy="-3.12031 0.1433 -2.84723" mid="0.0106955 -0.000462282 0.0331702" reflect="${reflect}" />
-      </xacro:if>
-      <xacro:unless value="$(arg use_capsule_collision)">
-        <collision>
-          <origin rpy="0 0 0" xyz="0 0 0"/>
-          <geometry>
-            <mesh filename="${MESH_PATH}/v2/hip_z_collision.stl" scale="1 ${reflect*1} 1"/>
-          </geometry>
-        </collision>
+      <xacro:unless value="${minimal_coll}">
+        <xacro:if value="$(arg use_capsule_collision)">
+          <xacro:capsule-collision e1="0.00653137 -0.00107636 0.0620231" e2="0.0148595 0.000151801 0.00431736" rad="0.10038884516307987" clen="0.058316498699378369" rpy="-3.12031 0.1433 -2.84723" mid="0.0106955 -0.000462282 0.0331702" reflect="${reflect}" />
+        </xacro:if>
+        <xacro:unless value="$(arg use_capsule_collision)">
+          <collision>
+            <origin rpy="0 0 0" xyz="0 0 0"/>
+            <geometry>
+              <mesh filename="${MESH_PATH}/v2/hip_z_collision.stl" scale="1 ${reflect*1} 1"/>
+            </geometry>
+          </collision>
+        </xacro:unless>
       </xacro:unless>
     </link>
@@ -115,14 +117,16 @@
         <material name="DarkGrey" />
       </visual>
-      <xacro:if value="$(arg use_capsule_collision)">
-        <xacro:capsule-collision e1="-0.0163525 -0.0136729 0.000327785" e2="-0.0177494 0.072721 0.00192874" rad="0.065228014094609946" clen="0.086420044518244921" rpy="-1.55227 -0.0161651 0.0158683" mid="-0.0170509 0.029524 0.00112826" reflect="${reflect}" />
-      </xacro:if>
-      <xacro:unless value="$(arg use_capsule_collision)">
-        <collision>
-          <origin xyz="0 0 0.0" rpy="0  0  0" />
-          <geometry>
-            <mesh filename="${MESH_PATH}/v2/hip_x_collision.stl" scale="1 ${reflect*1} 1"/>
-          </geometry>
-        </collision>
+      <xacro:unless value="${minimal_coll}">
+        <xacro:if value="$(arg use_capsule_collision)">
+          <xacro:capsule-collision e1="-0.0163525 -0.0136729 0.000327785" e2="-0.0177494 0.072721 0.00192874" rad="0.065228014094609946" clen="0.086420044518244921" rpy="-1.55227 -0.0161651 0.0158683" mid="-0.0170509 0.029524 0.00112826" reflect="${reflect}" />
+        </xacro:if>
+        <xacro:unless value="$(arg use_capsule_collision)">
+          <collision>
+            <origin xyz="0 0 0.0" rpy="0  0  0" />
+            <geometry>
+              <mesh filename="${MESH_PATH}/v2/hip_x_collision.stl" scale="1 ${reflect*1} 1"/>
+            </geometry>
+          </collision>
+        </xacro:unless>
       </xacro:unless>
     </link>
@@ -209,14 +213,16 @@
         <material name="Grey" />
       </visual>
-      <xacro:if value="$(arg use_capsule_collision)">
-        <xacro:capsule-collision e1="-0.0304137 0.105995 0.00632637" e2="0.00663845 -0.0117406 -0.00301129" rad="0.056285651716761462" clen="0.12378102303209611" rpy="1.64994 0.303997 0.32863" mid="-0.0118876 0.0471272 0.00165754" reflect="${reflect}" />
-      </xacro:if>
-      <xacro:unless value="$(arg use_capsule_collision)">
-        <collision>
-          <origin xyz="0 0 0.0" rpy="0 0 0" />
-          <geometry>
-            <mesh filename="${MESH_PATH}/v2/ankle_Y_collision.stl" scale="1 ${reflect*1} 1"/>
-          </geometry>
-        </collision>
+      <xacro:unless value="${minimal_coll}">
+        <xacro:if value="$(arg use_capsule_collision)">
+          <xacro:capsule-collision e1="-0.0304137 0.105995 0.00632637" e2="0.00663845 -0.0117406 -0.00301129" rad="0.056285651716761462" clen="0.12378102303209611" rpy="1.64994 0.303997 0.32863" mid="-0.0118876 0.0471272 0.00165754" reflect="${reflect}" />
+        </xacro:if>
+        <xacro:unless value="$(arg use_capsule_collision)">
+          <collision>
+            <origin xyz="0 0 0.0" rpy="0 0 0" />
+            <geometry>
+              <mesh filename="${MESH_PATH}/v2/ankle_Y_collision.stl" scale="1 ${reflect*1} 1"/>
+            </geometry>
+          </collision>
+        </xacro:unless>
       </xacro:unless>
     </link>

File: talos_description/urdf/talos_full_common.urdf.xacro (robot description, xacro)
@@ -17,4 +17,5 @@
   <xacro:arg name="gazebo_version" default="classic"/>
   <xacro:arg name="use_capsule_collision" default="false"/>
+  <xacro:arg name="minimal_coll" default="false"/>
   <xacro:arg name="disable_gazebo_camera" default="false"/>
   <xacro:arg name="include_gazebo" default="true"/>
@@ -89,6 +90,6 @@
                     disable_gazebo_camera="$(arg disable_gazebo_camera)"
                     head_type="$(arg head_type)"/>
-  <xacro:talos_arm name="arm" parent="torso_2_link" side="left" reflect="1"/>
-  <xacro:talos_arm name="arm" parent="torso_2_link" side="right" reflect="-1"/>
+  <xacro:talos_arm name="arm" parent="torso_2_link" side="left" reflect="1" minimal_coll="$(arg minimal_coll)"/>
+  <xacro:talos_arm name="arm" parent="torso_2_link" side="right" reflect="-1" minimal_coll="$(arg minimal_coll)"/>
   <xacro:ft_sensor name="wrist" parent="arm_right_7_link" side="right" reflect="1"  />
   <xacro:ft_sensor name="wrist" parent="arm_left_7_link"  side="left"  reflect="-1" />
@@ -97,6 +98,6 @@
     <xacro:talos_gripper name="gripper_right" parent="wrist_right_ft_tool_link" reflect="-1"/>
   </xacro:if>
-  <xacro:talos_leg prefix="left"  reflect="1" flexibility="$(arg flexibility)"/>
-  <xacro:talos_leg prefix="right" reflect="-1" flexibility="$(arg flexibility)"/>
+  <xacro:talos_leg prefix="left"  reflect="1" flexibility="$(arg flexibility)" minimal_coll="$(arg minimal_coll)"/>
+  <xacro:talos_leg prefix="right" reflect="-1" flexibility="$(arg flexibility)" minimal_coll="$(arg minimal_coll)"/>
   <xacro:talos_addons/>
   <xacro:if value="$(arg include_gazebo)">

File: talos_description/urdf/torso/torso.urdf.xacro (robot description, xacro)
@@ -61,14 +61,16 @@
         <material name="LightGrey" />
       </visual>
-      <xacro:if value="$(arg use_capsule_collision)">
-        <xacro:capsule-collision e1="-0.00232934 -0.0104948 -0.01235" e2="-0.00187524 0.0100705 -0.0118019" rad="0.091952314418329517" clen="0.020577608942189702" rpy="-1.54415 0.0220698 -0.0214895" mid="-0.00210229 -0.000212158 -0.0120759" />
-      </xacro:if>
-      <xacro:unless value="$(arg use_capsule_collision)">
-        <collision>
-          <origin xyz="0 0 0" rpy="0 0 0" />
-          <geometry>
-            <mesh filename="${MESH_PATH}/torso/torso_1.STL" scale="1 1 1"/>
-        </geometry>
-        </collision>
+      <xacro:unless value="$(arg minimal_coll)">
+        <xacro:if value="$(arg use_capsule_collision)">
+          <xacro:capsule-collision e1="-0.00232934 -0.0104948 -0.01235" e2="-0.00187524 0.0100705 -0.0118019" rad="0.091952314418329517" clen="0.020577608942189702" rpy="-1.54415 0.0220698 -0.0214895" mid="-0.00210229 -0.000212158 -0.0120759" />
+        </xacro:if>
+        <xacro:unless value="$(arg use_capsule_collision)">
+          <collision>
+            <origin xyz="0 0 0" rpy="0 0 0" />
+            <geometry>
+              <mesh filename="${MESH_PATH}/torso/torso_1.STL" scale="1 1 1"/>
+            </geometry>
+          </collision>
+        </xacro:unless>
       </xacro:unless>
     </link>
@@ -100,14 +102,16 @@
         <material name="LightGrey" />
       </visual>
-      <xacro:if value="$(arg use_capsule_collision)">
-        <xacro:capsule-collision e1="-0.0485657 0.111601 -0.05811" e2="-0.0490399 -0.110849 -0.0575714" rad="0.16382936354183916" clen="0.22245096803647357" rpy="1.56838 -0.00213179 -0.00212663" mid="-0.0488028 0.000376009 -0.0578407" />
-      </xacro:if>
-      <xacro:unless value="$(arg use_capsule_collision)">
-        <collision>
-          <origin xyz="0 0 0" rpy="0 0 0" />
-          <geometry>
-            <mesh filename="${MESH_PATH}/torso/base_link_collision.STL" scale="1 1 1"/>
-          </geometry>
-        </collision>
+      <xacro:unless value="$(arg minimal_coll)">
+        <xacro:if value="$(arg use_capsule_collision)">
+          <xacro:capsule-collision e1="-0.0485657 0.111601 -0.05811" e2="-0.0490399 -0.110849 -0.0575714" rad="0.16382936354183916" clen="0.22245096803647357" rpy="1.56838 -0.00213179 -0.00212663" mid="-0.0488028 0.000376009 -0.0578407" />
+        </xacro:if>
+        <xacro:unless value="$(arg use_capsule_collision)">
+          <collision>
+            <origin xyz="0 0 0" rpy="0 0 0" />
+            <geometry>
+              <mesh filename="${MESH_PATH}/torso/base_link_collision.STL" scale="1 1 1"/>
+            </geometry>
+          </collision>
+        </xacro:unless>
       </xacro:unless>
     </link>
