Commit message: disabling hip collisions (exploding on isaac)

File: talos_description/urdf/leg/leg.urdf.xacro (robot description, xacro)
@@ -150,14 +150,16 @@
         <material name="DarkGrey" />
       </visual>
-      <xacro:if value="$(arg use_capsule_collision)">
-        <xacro:capsule-collision e1="0.00475684 0.0387611 -0.305131" e2="0.0048036 0.0612963 -0.0132432" rad="0.14557912147210253" clen="0.29275626620252521" rpy="-0.077052 0.00015972 -6.15642e-06" mid="0.00478022 0.0500287 -0.159187" reflect="${reflect}" />
-      </xacro:if>
-      <xacro:unless value="$(arg use_capsule_collision)">
-        <collision>
-          <origin rpy="0 0 0" xyz="0 0 0"/>
-          <geometry>
-            <mesh filename="${MESH_PATH}/v2/hip_y_collision.stl" scale="1 ${reflect*1} 1"/>
-          </geometry>
-        </collision>
+      <xacro:unless value="${minimal_coll}">
+        <xacro:if value="$(arg use_capsule_collision)">
+          <xacro:capsule-collision e1="0.00475684 0.0387611 -0.305131" e2="0.0048036 0.0612963 -0.0132432" rad="0.14557912147210253" clen="0.29275626620252521" rpy="-0.077052 0.00015972 -6.15642e-06" mid="0.00478022 0.0500287 -0.159187" reflect="${reflect}" />
+        </xacro:if>
+        <xacro:unless value="$(arg use_capsule_collision)">
+          <collision>
+            <origin rpy="0 0 0" xyz="0 0 0"/>
+            <geometry>
+              <mesh filename="${MESH_PATH}/v2/hip_y_collision.stl" scale="1 ${reflect*1} 1"/>
+            </geometry>
+          </collision>
+        </xacro:unless>
       </xacro:unless>
     </link>

Commit message: added sphere collisions for feet

File: talos_description/urdf/leg/leg.urdf.xacro (robot description, xacro)
@@ -262,4 +262,26 @@
     <link name="${prefix}_sole_link">
       <xacro:call macro="${prefix}_sole_link_inertial" />
+      <xacro:if value="$(arg foot_corner_spheres)">
+        <xacro:property name="foot_corner_radius" value="$(arg foot_corner_sphere_radius)" />
+        <xacro:property name="foot_corner_x" value="$(arg foot_corner_sphere_x)" />
+        <xacro:property name="foot_corner_y" value="$(arg foot_corner_sphere_y)" />
+        <xacro:property name="foot_corner_z" value="$(arg foot_corner_sphere_z)" />
+        <collision>
+          <origin xyz="${foot_corner_x} ${foot_corner_y} ${foot_corner_z}" rpy="0 0 0" />
+          <geometry><sphere radius="${foot_corner_radius}" /></geometry>
+        </collision>
+        <collision>
+          <origin xyz="${foot_corner_x} ${-foot_corner_y} ${foot_corner_z}" rpy="0 0 0" />
+          <geometry><sphere radius="${foot_corner_radius}" /></geometry>
+        </collision>
+        <collision>
+          <origin xyz="${-foot_corner_x} ${foot_corner_y} ${foot_corner_z}" rpy="0 0 0" />
+          <geometry><sphere radius="${foot_corner_radius}" /></geometry>
+        </collision>
+        <collision>
+          <origin xyz="${-foot_corner_x} ${-foot_corner_y} ${foot_corner_z}" rpy="0 0 0" />
+          <geometry><sphere radius="${foot_corner_radius}" /></geometry>
+        </collision>
+      </xacro:if>
     </link>
     <joint name="leg_${prefix}_sole_fix_joint" type="fixed">

File: talos_description/urdf/talos_full_common.urdf.xacro (robot description, xacro)
@@ -18,4 +18,9 @@
   <xacro:arg name="use_capsule_collision" default="false"/>
   <xacro:arg name="minimal_coll" default="false"/>
+  <xacro:arg name="foot_corner_spheres" default="false"/>
+  <xacro:arg name="foot_corner_sphere_radius" default="0.005"/>
+  <xacro:arg name="foot_corner_sphere_x" default="0.103"/>
+  <xacro:arg name="foot_corner_sphere_y" default="0.063"/>
+  <xacro:arg name="foot_corner_sphere_z" default="-0.001"/>
   <xacro:arg name="disable_gazebo_camera" default="false"/>
   <xacro:arg name="include_gazebo" default="true"/>
